File: Design/micromouse/sensor.brd (EAGLE design)
At the start: 160 x 100 mm, 9 parts

Commit message: add firmware
Parts:
- removed C2: 10u/16v, rcl:C0603
- removed JP1: (no value), pinhead:1X03/90
- added C3, C4, C5: 0.1u/16v, rcl:C0603
- added JP2: (no value), pinhead:1X04/90
- added R4: 330, rcl:R0603
- added R5: 22, rcl:R0603
- R3: value 330 -> 22
- moved R3 45.0 mm to (3.81, 6.35), flipped to the bottom, turned to 180 degrees
- moved R2 44.1 mm to (7.62, 11.4), flipped to the bottom, turned to 90 degrees
- moved LED3 43.1 mm to (12.6, 7.62), turned to 90 degrees
- moved R1 37.8 mm to (10.2, 6.35), flipped to the bottom, turned to 90 degrees
- moved C1 37.2 mm to (11.4, 2.54), flipped to the bottom
- moved LED2 34.3 mm to (3.81, 3.81)
- moved LED1 28.7 mm to (3.81, 11.4)
Connections:
- removed net N$2: C2.2, JP1.2, LED1.K, LED2.K, R1.2, R2.2
- removed net N$3: C1.1, JP1.1, R3.2
- new net GND: C3.2, C5.2, JP2.2, LED1.K, LED2.K, R1.2, R2.2, R4.2
- new net N$10: C4.2, R4.1, R5.2
- new net SENSOR: C5.1, JP2.3, R5.1
- new net V+: JP2.4, LED3.A
- new net VCC: C1.1, JP2.1
- net N$1: now also C3.1, R3.1; no longer C1.2, R1.1
- net N$4: now also C4.1
- net N$5: now also C1.2, R1.1, R3.2; no longer C2.1, LED3.A, R3.1
Routing:
- net N$1: track 0.00 -> 16.6 mm
- net N$5: track 0.00 -> 15.3 mm
- net N$4: track 0.00 -> 14.2 mm, vias 0 -> 2
- net SENSOR: track 0.00 -> 8.81 mm
- net N$10: track 0.00 -> 7.54 mm, vias 0 -> 1
- net V+: track 0.00 -> 3.41 mm
- net VCC: track 0.00 -> 2.96 mm
- added copper zone on layer 1, net GND
- added copper zone on layer 16, net GND
Other:
- board size 160 x 100 mm -> 20 x 15 mm
