File: Design/micromouse/mouse.brd (EAGLE design)
At the start: 50 x 50 mm, 73 parts, among them IC1 LPC1549JBD48, IC2 DRV8848PWPR, IC3 TLV61048DBVT, IC4 TPD4S014DSQR, J1 B2B-XH-A(LF)(SN), J10 SM04B-ZESS-TB(LF)(SN), J11 SM04B-ZESS-TB(LF)(SN), J12 SM04B-ZESS-TB(LF)(SN), J2 B2B-XH-A(LF)(SN), J3 B2B-XH-A(LF)(SN), J4 J_USB_MICROAB_HIROSE_ZX62-AB-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, J8 SM06B-ZESS-TB(LF)(SN), J9 SM06B-ZESS-TB(LF)(SN), U1 ADR5041, U2 MCP1700T-33, Y1 FA238V

Commit message: add firmware
Parts:
- added SV1: (no value), con-lstb:MA03-1
- moved J10 1.27 mm to (45.7, 38.1)
- moved J11 1.27 mm to (45.7, 24.8)
- moved J12 1.27 mm to (45.7, 11.4)
- moved R27 0.77 mm to (35.1, 16.9)
- moved R25 0.76 mm to (35.1, 40.6)
- moved R26 0.76 mm to (35.1, 29.2)
- moved C1 0.51 mm to (23.6, 8.89)
- moved C2 0.51 mm to (17.0, 8.89)
Connections:
- net GND: now also SV1.3
- net U0RX: now also SV1.2
- net U0TX: now also SV1.1
Routing:
- net U0RX: track 0.00 -> 15.4 mm, vias 0 -> 1
- net U0TX: track 0.00 -> 15.1 mm, vias 0 -> 1
- net V+: track 63.9 -> 65.8 mm
- net !SENSOR1: track 70.7 -> 71.9 mm
- net !SENSOR3: track 32.9 -> 34.2 mm, vias 7 -> 6
- net !SENSOR2: track 61.0 -> 62.3 mm
- net !ISP1: track 10.0 -> 11.0 mm
- net N$26: track 11.5 -> 12.3 mm
- net N$31: track 15.5 -> 16.2 mm
- net N$22: track 2.30 -> 1.54 mm
- net N$24: track 15.0 -> 15.7 mm
- net N$1: track 4.95 -> 5.47 mm
- net N$2: track 5.87 -> 5.36 mm
- net GND: vias 52 -> 53

Commit message: circuit design
Parts:
- removed D5: (no value), MotorDriver:DIODE_SOD523
- removed IC3: TLV61048DBVT, TLV61048DBVT:SOT95P280X145-6N
- removed L1: NR50404R7N, NR5040T330M:NR5040T2R2N
- removed LED2: (no value), MotorDriver:LED1608
- removed R14: 1k, rcl:R0603
- removed R7: (no value), rcl:R0603
- removed R8: 80k, rcl:R0603
- removed R9: 10k, rcl:R0603
- added D4: (no value), MotorDriver:DIODE_SOD523
- added IC5: NCP1117LPST50T3G, NCP1117LPST50T3G:SOT230P700X180-4N
- C5: value 0.1u/16v -> 1u/16v
- C6: value 1u/6.3v -> 1u/16v
- C7: value 10u/16v -> 1u/6.3v
- D1, D3: device diode:DO214AC -> diode:SMB
- moved D1 39.2 mm to (2.29, 4.45), flipped to the top, turned to 270 degrees
- moved C5 17.4 mm to (18.7, 40.9), turned to 0 degrees
- moved T3 15.8 mm to (37.3, 8.26), turned to 0 degrees
- moved C6 15.0 mm to (26.3, 38.4), turned to 180 degrees
- moved T2 7.04 mm to (34.5, 21.1), turned to 180 degrees
- moved T1 5.58 mm to (33.7, 26.8), turned to 180 degrees
- moved C7 3.86 mm to (25.4, 27.9), turned to 180 degrees
- moved D3 1.09 mm to (26.3, 41.3)
- moved R22 0.92 mm to (32.8, 36.1)
Connections:
- removed net N$16: IC3.3, R8.2, R9.1
- removed net N$17: LED2.K, R14.1
- removed net N$18: C6.1, C8.1, D2.K, D3.C, D5.K, IC3.5, L1.1, U2.3
- removed net N$27: R23.1, T2.2
- removed net N$28: R24.1, T3.2
- removed net N$7: D1.A, IC3.1, L1.2
- removed net VMEN: IC1.43, IC3.4, R7.1
- new net N$30: J10.2, T1.1
- new net N$32: J11.2, T2.1
- new net N$33: J12.2, T3.1
- net +5V: now also C7.1, C8.1, D1.C, D2.K, D4.A, IC5.2, IC5.4, J10.4, J11.4, J12.4, R22.1, R23.1, R24.1, U2.3; no longer D5.A, IC4.1, IC4.2
- net GND: now also IC5.1, T1.2, T2.2, T3.2; no longer IC3.2, J10.2, J11.2, J12.2, R14.2, R7.2, R9.2
- net N$6: now also D1.A, IC4.1, IC4.2; no longer R22.1, T1.2
- net V+: now also C6.1, D3.C, D4.K, IC5.3; no longer C7.1, D1.C, J10.4, J11.4, J12.4, LED2.A, R8.1, T1.1, T2.1, T3.1
Routing:
- net +5V: track 7.10 -> 262.5 mm, vias 0 -> 8
- net N$18: track 188.1 -> 0.00 mm, vias 7 -> 0
- net V+: track 65.8 -> 100.5 mm, vias 8 -> 5
- net VMEN: track 34.6 -> 0.00 mm, vias 4 -> 0
- net N$16: track 33.3 -> 0.00 mm, vias 4 -> 0
- net N$30: track 0.00 -> 16.5 mm, vias 0 -> 1
- net N$7: track 14.7 -> 0.00 mm
- net +3V3: track 325.0 -> 338.5 mm, vias 15 -> 14
- net N$32: track 0.00 -> 8.69 mm, vias 0 -> 1
- net N$27: track 8.28 -> 0.00 mm
- net N$33: track 0.00 -> 6.58 mm, vias 0 -> 1
- net N$28: track 5.35 -> 0.00 mm
- net SENSOR_EN: track 37.2 -> 32.3 mm, vias 3 -> 4
- net N$6: track 4.67 -> 8.52 mm
- net N$17: track 2.13 -> 0.00 mm
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- removed copper zone on layer 16, net +3V3
- removed copper zone on layer 1, net V+
- removed copper zone on layer 16, net V+
