File: Design/micromouse/mouse.sch (EAGLE design)
At the start: 73 parts, among them IC1 LPC1549JBD48, IC2 DRV8848PWPR, IC3 TLV61048DBVT, IC4 TPD4S014DSQR, J1 B2B-XH-A(LF)(SN), J10 SM04B-ZESS-TB(LF)(SN), J11 SM04B-ZESS-TB(LF)(SN), J12 SM04B-ZESS-TB(LF)(SN), J2 B2B-XH-A(LF)(SN), J3 B2B-XH-A(LF)(SN), J4 J_USB_MICROAB_HIROSE_ZX62-AB-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, J8 SM06B-ZESS-TB(LF)(SN), J9 SM06B-ZESS-TB(LF)(SN), U1 ADR5041, U2 MCP1700T-33, Y1 FA238V

Commit message: add firmware
Parts:
- added SV1: (no value), con-lstb:MA03-1
Connections:
- net GND: now also SV1.3
- net U0RX: now also SV1.2
- net U0TX: now also SV1.1
Changed lines of the file:
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@@
 <part name="SUPPLY7" library="supply2" library_urn="urn:adsk.eagle:library:372" deviceset="V+" device=""/>
 <part name="SUPPLY8" library="supply2" library_urn="urn:adsk.eagle:library:372" deviceset="V+" device=""/>
+<part name="SV1" library="con-lstb" library_urn="urn:adsk.eagle:library:162" deviceset="MA03-1" device="" package3d_urn="urn:adsk.eagle:package:8339/1"/>
+<part name="GND40" library="supply1" library_urn="urn:adsk.eagle:library:371" deviceset="GND" device=""/>
 </parts>
 <sheets>
@@
 <attribute name="VALUE" x="400.05" y="85.09" size="1.778" layer="96"/>
 </instance>
+<instance part="SV1" gate="G$1" x="421.64" y="106.68" smashed="yes" rot="R180">
+<attribute name="VALUE" x="422.91" y="114.3" size="1.778" layer="96" rot="R180"/>
+<attribute name="NAME" x="422.91" y="100.838" size="1.778" layer="95" rot="R180"/>
+</instance>
+<instance part="GND40" gate="1" x="411.48" y="93.98" smashed="yes">
+<attribute name="VALUE" x="408.94" y="91.44" size="1.778" layer="96"/>
+</instance>
 </instances>
 <busses>
@@
 <wire x1="144.78" y1="71.12" x2="144.78" y2="48.26" width="0.1524" layer="91"/>
 <pinref part="GND39" gate="1" pin="GND"/>
+</segment>
+<segment>
+<pinref part="SV1" gate="G$1" pin="3"/>
+<wire x1="414.02" y1="104.14" x2="411.48" y2="104.14" width="0.1524" layer="91"/>
+<wire x1="411.48" y1="104.14" x2="411.48" y2="96.52" width="0.1524" layer="91"/>
+<pinref part="GND40" gate="1" pin="GND"/>
 </segment>
 </net>
@@
 <label x="81.28" y="22.86" size="1.27" layer="95" rot="R270" xref="yes"/>
 </segment>
+<segment>
+<pinref part="SV1" gate="G$1" pin="2"/>
+<wire x1="414.02" y1="106.68" x2="408.94" y2="106.68" width="0.1524" layer="91"/>
+<label x="408.94" y="106.68" size="1.27" layer="95" rot="R180" xref="yes"/>
+</segment>
 </net>
 <net name="U0TX" class="0">
@@
 <label x="83.82" y="22.86" size="1.27" layer="95" rot="R270" xref="yes"/>
 </segment>
-</net>
+<segment>
+<pinref part="SV1" gate="G$1" pin="1"/>
+<wire x1="414.02" y1="109.22" x2="408.94" y2="109.22" width="0.1524" layer="91"/>
+<label x="408.94" y="109.22" size="1.27" layer="95" rot="R180" xref="yes"/>
+</segment>
+</net>

Commit message: circuit design
Parts:
- removed D5: (no value), MotorDriver:SBD-SOD523
- removed IC3: TLV61048DBVT, TLV61048DBVT:TLV61048DBVT
- removed L1: NR50404R7N, NR5040T330M:NR5040T330M
- removed LED2: (no value), MotorDriver:LED1608
- removed R14: 1k, rcl:R-US_R0603
- removed R7: (no value), rcl:R-US_R0603
- removed R8: 80k, rcl:R-US_R0603
- removed R9: 10k, rcl:R-US_R0603
- added D4: (no value), MotorDriver:SBD-SOD523
- added IC5: NCP1117LPST50T3G, NCP1117LPST50T3G:NCP1117LPST50T3G
- C5: value 0.1u/16v -> 1u/16v
- C6: value 1u/6.3v -> 1u/16v
- C7: value 10u/16v -> 1u/6.3v
- D1, D3: device diode:DIODE-DO214AC -> diode:DIODE-SMB
Connections:
- removed net N$16: IC3.FB, R8.2, R9.1
- removed net N$17: LED2.K, R14.1
- removed net N$18: C6.1, C8.1, D2.K, D3.C, D5.K, IC3.VIN, L1.1, U2.VI
- removed net N$27: R23.1, T2.S
- removed net N$28: R24.1, T3.S
- removed net N$7: D1.A, IC3.SW, L1.2
- removed net VMEN: IC1.PIO0_24/SCTO_OUT6, IC3.EN, R7.1
- new net N$30: J10.2, T1.D
- new net N$32: J11.2, T2.D
- new net N$33: J12.2, T3.D
- net +5V: now also C7.1, C8.1, D1.C, D2.K, D4.A, IC5.OUT_1, J10.4, J11.4, J12.4, R22.1, R23.1, R24.1, U2.VI; no longer D5.A, IC4.VBUSOUT
- net GND: now also IC5.ADJ/GND, T1.S, T2.S, T3.S; no longer IC3.GND, J10.2, J11.2, J12.2, R14.2, R7.2, R9.2
- net N$6: now also D1.A, IC4.VBUSOUT; no longer R22.1, T1.S
- net V+: now also C6.1, D3.C, D4.K, IC5.IN; no longer C7.1, D1.C, J10.4, J11.4, J12.4, LED2.A, R8.1, T1.D, T2.D, T3.D
Other:
- note added: "LiPO 2Cell 7.4V-8.4V"
- note removed: "LiPO 1Cell 3.7V-4.2V"
- note removed: "Vout=7.2[V]"
- moved on the sheet: C5, C6, C7, D1, T1, T2, T3
